File: PCB_Health.V2.kicad_pcb (KiCad board)
At the start: 2 copper layers, 173.5 x 96 mm, 53 parts, among them J1 Conn_01x02_Socket, J2 Conn_01x02_Socket, J3 Conn_01x04_Socket, J4 Conn_01x04_Socket, J5 Conn_01x02_Socket, K1 RT424012, Q1 BC337, U1 H11L1, U2 MAX6675ISA_, U3 MAX6675ISA_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

Commit message: Creating Fab and assy outputs for PCB_Health board
Parts:
- added J6: Conn_01x03_Pin, Connector_Molex:Molex_KK-254_AE-6410-03A_1x03_P2.54mm_Vertical, F.Cu at (184.4, 50.6)
- C8: footprint Capacitor_THT:C_Disc_D9.0mm_W5.0mm_P5.00mm -> Capacitor_SMD:C_1210_3225Metric
- D1: value 1N4148 -> 1N4001; footprint Diode_THT:D_DO-35_SOD27_P7.62mm_Horizontal -> Diode_THT:D_DO-41_SOD81_P10.16mm_Horizontal
- F4: value 2A -> 3A
- J3, J4: footprint Connector_PinHeader_2.54mm:PinHeader_1x04_P2.54mm_Vertical -> Connector_Molex:Molex_KK-254_AE-6410-04A_1x04_P2.54mm_Vertical
- moved R3 6.18 mm to (189.2, 86.4), turned to -90 degrees
- moved D1 2.87 mm to (150.7, 96.5)
- moved C8 1.98 mm to (110.2, 90.0)
- turned J3 to 180 degrees
- turned J4 to 180 degrees
Connections:
- A1 pad 19: unconnected-(A1-GPIO36-Pad19) -> /GPIO36
- A1 pad 20: unconnected-(A1-GPIO39-Pad20) -> /GPIO39
Routing:
- net /GPIO36: track 0.00 -> 46.8 mm
- net /GPIO39: track 0.00 -> 42.5 mm
- net Net-(D1-A): track 37.6 -> 17.6 mm
- net /GPIO33: track 24.3 -> 10.9 mm
- net GND: track 15.8 -> 26.8 mm, vias 0 -> 1
- net Net-(J3-Pin_1): track 162.9 -> 169.5 mm
- net +5V: track 350.0 -> 355.1 mm
- net Net-(R3-Pad1): track 8.39 -> 3.86 mm
- net +12V: track 177.6 -> 180.5 mm
- net Net-(D2-K): track 63.5 -> 66.3 mm
- net /GPIO32: track 64.5 -> 67.0 mm
- net /GPIO3: track 75.5 -> 76.3 mm
- net /GPIO5: track 73.9 -> 73.2 mm
- added copper zone on In1.Cu, net GND
- added copper zone on In2.Cu, net GND
Other:
- copper layers 2 -> 4
- board text added: "I2C"
